Commit message: fix: Fix the incorrect translation direction issue in Gazebo simulation

File: agv_pro_description/urdf/robot/wheel_macro.urdf.xacro (robot description, xacro)
@@ -17,5 +17,5 @@
       <xacro:property name="mesh" value="file://$(find agv_pro_description)/meshes/wheel_lf_link.stl" />
       <xacro:property name="visual_rotation" value="${pi}" />
-      <xacro:property name="fdir" value="1.0 -1.0 0.0" />
+      <xacro:property name="fdir" value="1.0 1.0 0.0" />
     </xacro:if>
     <!-- 前右轮 -->
@@ -25,5 +25,5 @@
       <xacro:property name="mesh" value="file://$(find agv_pro_description)/meshes/wheel_rf_link.stl" />
       <xacro:property name="visual_rotation" value="${pi}" />
-      <xacro:property name="fdir" value="1.0 1.0 0.0" />
+      <xacro:property name="fdir" value="1.0 -1.0 0.0" />
     </xacro:if>
     <!-- 后左轮 -->
@@ -33,5 +33,5 @@
       <xacro:property name="mesh" value="file://$(find agv_pro_description)/meshes/wheel_lb_link.stl" />
       <xacro:property name="visual_rotation" value="${0.0}" />
-      <xacro:property name="fdir" value="1.0 1.0 0.0" />
+      <xacro:property name="fdir" value="1.0 -1.0 0.0" />
     </xacro:if>
     <!-- 后右轮 -->
@@ -41,5 +41,5 @@
       <xacro:property name="mesh" value="file://$(find agv_pro_description)/meshes/wheel_rb_link.stl" />
       <xacro:property name="visual_rotation" value="${0.0}" />
-      <xacro:property name="fdir" value="1.0 -1.0 0.0" />
+      <xacro:property name="fdir" value="1.0 1.0 0.0" />
     </xacro:if>
     <joint name="${side}_wheel_joint" type="continuous">
